Commit message: last

File: hydrone_aerial_underwater_description/urdf/hydrone_aerial_underwater_aerial.gazebo.xacro (robot description, xacro)
@@ -11,5 +11,5 @@
     <!-- <xacro:property name="volume" value="0.00001"/> -->
     <!-- <xacro:property name="volume" value="0.001"/> -->
-    <xacro:property name="volume" value="0.0001"/>
+    <xacro:property name="volume" value="0.00005"/>
     <!-- <xacro:property name="volume" value="0.00005"/> -->
     <xacro:property name="M_PI" value="3.1415926535897931" />
@@ -35,18 +35,18 @@
                 </added_mass>
                 <linear_damping>
-                    0.0125   0.0         0.0         0.0         0.0         0.0
-                    0.0         0.0125   0.0         0.0         0.0         0.0
-                    0.0         0.0         0.0499   0.0         0.0         0.0
-                    0.0         0.0         0.0         0.0125   0.0         0.0
-                    0.0         0.0         0.0         0.0         0.0125   0.0
-                    0.0         0.0         0.0         0.0         0.0         0.0499
+                    -10.0125   0.0         0.0         0.0         0.0         0.0
+                    0.0         -10.0125   0.0         0.0         0.0         0.0
+                    0.0         0.0         -10.0499   0.0         0.0         0.0
+                    0.0         0.0         0.0         -1.0125   0.0         0.0
+                    0.0         0.0         0.0         0.0         -1.0125   0.0
+                    0.0         0.0         0.0         0.0         0.0         -1.0499
                 </linear_damping>
                 <quadratic_damping>
-                    0.0125   0.0         0.0         0.0         0.0         0.0
-                    0.0         0.0125   0.0         0.0         0.0         0.0
-                    0.0         0.0         0.0499   0.0         0.0         0.0
-                    0.0         0.0         0.0         0.0125   0.0         0.0
-                    0.0         0.0         0.0         0.0         0.0125   0.0
-                    0.0         0.0         0.0         0.0         0.0         0.0499
+                    -10.0125   0.0         0.0         0.0         0.0         0.0
+                    0.0         -10.0125   0.0         0.0         0.0         0.0
+                    0.0         0.0         -10.0499   0.0         0.0         0.0
+                    0.0         0.0         0.0         -1.0125   0.0         0.0
+                    0.0         0.0         0.0         0.0         -1.0125   0.0
+                    0.0         0.0         0.0         0.0         0.0         -1.0499
                 </quadratic_damping>
                 <!-- Added mass: see p.28 in Berg2012 -->
