Commit message: mp multi

File: hydrone_aerial_underwater_description/urdf/hydrone_aerial_underwater_base_aerial.xacro (robot description, xacro)
@@ -83,203 +83,14 @@
       <xacro:insert_block name="body_inertia" />
     </xacro:multirotor_base_macro>
-    <!-- <joint name="${namespace}/thruster_1_joint" type="continuous">
-      <origin xyz="0.19725 -0.19725 -0.055" rpy="0 0 0"/>
-      <axis xyz="0 0 1"/>
-      <parent link="${namespace}/base_link"/>
-      <child link="${namespace}/thruster_1"/>
-    </joint>
-    <link name="${namespace}/thruster_1">
-      <xacro:box_inertial x="0" y="0" z="0" mass="0.1">
-        <origin xyz="0 0 0" rpy="0 0 0"/>
-      </xacro:box_inertial>
-      <visual>
-        <origin xyz="-0.03 -0.0315 -0.01" rpy="0 0 0"/>
-        <geometry>
-          <mesh filename="file://$(find hydrone_aerial_underwater_description)/meshes/aquatic_propeller_1.dae" scale="1 1 1"/>
-        </geometry>
-      </visual>
-      <collision>
-        <origin xyz="0.0 0.0 0.0" rpy="0 0 0"/>
-        <geometry>
-          <box size="0.06 0.06 0.04"/>
-        </geometry>
-      </collision>
-    </link>
-    <gazebo>
-      <plugin name="${namespace}_0_thruster_model" filename="libuuv_thruster_ros_plugin.so">
-        <linkName>${namespace}/thruster_1</linkName>
-        <jointName>${namespace}/thruster_1_joint</jointName>
-        <thrusterID>1</thrusterID>
-        <gain>1</gain>
-        <clampMax>-3000</clampMax>
-        <clampMin>3000</clampMin>
-        <thrustMin>-1000</thrustMin>
-        <thrustMax>1000</thrustMax>
-        <thrust_efficiency>1</thrust_efficiency>
-        <propeller_efficiency>1</propeller_efficiency>
-        <dynamics>
-          <type>FirstOrder</type>
-          <timeConstant>0.05</timeConstant>
-        </dynamics>
-        <conversion>
-          <type>Basic</type>
-          <rotorConstant>0.00031</rotorConstant>
-        </conversion>
-      </plugin>
-    </gazebo>
-    <gazebo reference="${namespace}/thruster_1">
-      <selfCollide>false</selfCollide>
-      <material>Gazebo/Blue</material>
-    </gazebo>
-    <joint name="${namespace}/thruster_2_joint" type="continuous">
-      <origin xyz="0.19725 0.19725 -0.055" rpy="0 0 0"/>
-      <axis xyz="0 0 -1"/>
-      <parent link="${namespace}/base_link"/>
-      <child link="${namespace}/thruster_2"/>
-    </joint>
-    <link name="${namespace}/thruster_2">
-      <xacro:box_inertial x="0" y="0" z="0" mass="0.1">
-        <origin xyz="0 0 0" rpy="0 0 0"/>
-      </xacro:box_inertial>
-      <collision>
-        <origin xyz="-0.0 -0.0 -0.0" rpy="0 0 0"/>
-        <geometry>
-          <box size="0.06 0.06 0.04"/>
-        </geometry>
-      </collision>
-      <visual>
-        <origin xyz="-0.03 -0.0315 -0.01" rpy="0 0 0"/>
-        <geometry>
-          <mesh filename="file://$(find hydrone_aerial_underwater_description)/meshes/aquatic_propeller.dae" scale="1 1 1"/>
-        </geometry>
-      </visual>
-    </link>
-    <gazebo>
-      <plugin name="${namespace}_2_thruster_model" filename="libuuv_thruster_ros_plugin.so">
-        <linkName>${namespace}/thruster_2</linkName>
-        <jointName>${namespace}/thruster_2_joint</jointName>
-        <thrusterID>2</thrusterID>
-        <gain>1</gain>
-        <clampMax>-3000</clampMax>
-        <clampMin>3000</clampMin>
-        <thrustMin>-1000</thrustMin>
-        <thrustMax>1000</thrustMax>
-        <thrust_efficiency>1</thrust_efficiency>
-        <propeller_efficiency>1</propeller_efficiency>
-        <dynamics>
-          <type>FirstOrder</type>
-          <timeConstant>0.05</timeConstant>
-        </dynamics>
-        <conversion>
-          <type>Basic</type>
-          <rotorConstant>0.00031</rotorConstant>
-        </conversion>
-      </plugin>
-    </gazebo>
-    <gazebo reference="${namespace}/thruster_2">
-      <selfCollide>false</selfCollide>
-      <material>Gazebo/Blue</material>
-    </gazebo>
-    <joint name="${namespace}/thruster_3_joint" type="continuous">
-      <origin xyz="-0.19725 0.19725 -0.055" rpy="0 0 0"/>
-      <axis xyz="0 0 1"/>
-      <parent link="${namespace}/base_link"/>
-      <child link="${namespace}/thruster_3"/>
-    </joint>
-    <link name="${namespace}/thruster_3">
-      <xacro:box_inertial x="0" y="0" z="0" mass="0.1">
-        <origin xyz="0 0 0" rpy="0 0 0"/>
-      </xacro:box_inertial>
-      <collision>
-        <origin xyz="-0.0 -0.0 -0.0" rpy="0 0 0"/>
-        <geometry>
-          <box size="0.06 0.06 0.04"/>
-        </geometry>
-      </collision>
-      <visual>
-        <origin xyz="-0.03 -0.0315 -0.01" rpy="0 0 0"/>
-        <geometry>
-          <mesh filename="file://$(find hydrone_aerial_underwater_description)/meshes/aquatic_propeller_1.dae" scale="1 1 1"/>
-        </geometry>
-      </visual>
-    </link>
-    <gazebo>
-      <plugin name="${namespace}_3_thruster_model" filename="libuuv_thruster_ros_plugin.so">
-        <linkName>${namespace}/thruster_3</linkName>
-        <jointName>${namespace}/thruster_3_joint</jointName>
-        <thrusterID>3</thrusterID>
-        <gain>1</gain>
-        <clampMax>-3000</clampMax>
-        <clampMin>3000</clampMin>
-        <thrustMin>-1000</thrustMin>
-        <thrustMax>1000</thrustMax>
-        <thrust_efficiency>1</thrust_efficiency>
-        <propeller_efficiency>1</propeller_efficiency>
-        <dynamics>
-          <type>FirstOrder</type>
-          <timeConstant>0.05</timeConstant>
-        </dynamics>
-        <conversion>
-          <type>Basic</type>
-          <rotorConstant>0.00031</rotorConstant>
-        </conversion>
-      </plugin>
-    </gazebo>
-    <gazebo reference="${namespace}/thruster_3">
-      <selfCollide>false</selfCollide>
-      <material>Gazebo/Blue</material>
-    </gazebo>
-    <joint name="${namespace}/thruster_4_joint" type="continuous">
-      <origin xyz="-0.19725 -0.19725 -0.055" rpy="0 0 0"/>
-      <axis xyz="0 0 -1"/>
-      <parent link="${namespace}/base_link"/>
-      <child link="${namespace}/thruster_4"/>
-    </joint>
-    <link name="${namespace}/thruster_4">
-      <xacro:box_inertial x="0" y="0" z="0" mass="0.1">
-        <origin xyz="0 0 0" rpy="0 0 0"/>
-      </xacro:box_inertial>
-      <collision>
-        <origin xyz="-0.0 -0.0 -0.0" rpy="0 0 0"/>
-        <geometry>
-          <box size="0.06 0.06 0.04"/>
-        </geometry>
-      </collision>
-      <visual>
-        <origin xyz="-0.03 -0.0315 -0.01" rpy="0 0 0"/>
-        <geometry>
-          <mesh filename="file://$(find hydrone_aerial_underwater_description)/meshes/aquatic_propeller.dae" scale="1 1 1"/>
-        </geometry>
-      </visual>
-    </link>
-    <gazebo>
-      <plugin name="${namespace}_4_thruster_model" filename="libuuv_thruster_ros_plugin.so">
-        <linkName>${namespace}/thruster_4</linkName>
-        <jointName>${namespace}/thruster_4_joint</jointName>
-        <thrusterID>4</thrusterID>
-        <gain>1</gain>
-        <clampMax>-3000</clampMax>
-        <clampMin>3000</clampMin>
-        <thrustMin>-1000</thrustMin>
-        <thrustMax>1000</thrustMax>
-        <thrust_efficiency>1</thrust_efficiency>
-        <propeller_efficiency>1</propeller_efficiency>
-        <dynamics>
-          <type>FirstOrder</type>
-          <timeConstant>0.05</timeConstant>
-        </dynamics>
-        <conversion>
-          <type>Basic</type>
-          <rotorConstant>0.00031</rotorConstant>
-        </conversion>
-      </plugin>
-    </gazebo>
-    <gazebo reference="${namespace}/thruster_4">
-      <selfCollide>false</selfCollide>
-      <material>Gazebo/Blue</material>
-    </gazebo> -->
-    <gazebo reference="${namespace}/base_link">
-      <material>Gazebo/White</material>
-    </gazebo>
+    <xacro:if value="${use_simplified_mesh}">
+      <gazebo reference="${namespace}/base_link">
+        <material>Gazebo/Gold</material>
+      </gazebo>
+    </xacro:if>
+    <xacro:unless value="${use_simplified_mesh}">
+      <gazebo reference="${namespace}/base_link">
+        <material>Gazebo/White</material>
+      </gazebo>
+    </xacro:unless>
     <!-- Instantiate rotors -->
     <xacro:vertical_rotor
@@ -432,32 +243,4 @@
     <!-- <xacro:include filename="$(find hydrone_aerial_underwater_description)/urdf/hydrone_aerial_underwater_actuators.xacro" /> -->
   </xacro:macro>
-  <!-- <joint name="scan_joint" type="fixed">
-    <parent link="${namespace}/base_link"/>
-    <child link="base_scan"/>
-    <origin xyz="0.0 0 -0.1" rpy="0 0 0"/>
-  </joint>
-  <link name="base_scan">
-    <visual>
-      <origin xyz="0 0 0.0" rpy="0 0 0"/>
-      <geometry>
-        <box size="0.01 0.01 0.01"/>
-      </geometry>
-      <material name="dark"/>
-    </visual>
-    <collision>
-      <origin xyz="0 0 0.0" rpy="0 0 0"/>
-      <geometry>
-        <box size="0.01 0.01 0.01"/>
-      </geometry>
-      <material name="dark"/>
-    </collision>
-    <inertial>
-      <mass value="0.114" />
-      <origin xyz="0 0 0" />
-      <inertia ixx="0.001" ixy="0.0" ixz="0.0"
-              iyy="0.001" iyz="0.0"
-              izz="0.001" />
-    </inertial>
-  </link> -->
   <joint name="scan_joint" type="fixed">
     <parent link="${namespace}/base_link"/>
@@ -487,403 +270,3 @@
     </inertial>
   </link>
-  <!-- <joint name="ir_front_joint_0" type="fixed">
-    <axis xyz="0 1 0" />
-    <origin rpy="0 0 0" xyz="0.02 0 0.1" />
-    <parent link="${namespace}/base_link"/>
-    <child link="base_ir_front_0"/>
-  </joint>
-  <link name="base_ir_front_0">
-    <collision>
-      <origin xyz="0 0 0" rpy="0 0 0"/>
-      <geometry>
-        <box size="0.01 0.01 0.01"/>
-      </geometry>
-    </collision>
-    <visual>
-      <origin xyz="0 0 0" rpy="0 0 0"/>
-      <geometry>
-        <box size="0.01 0.01 0.01"/>
-      </geometry>
-    </visual>
-    <inertial>
-      <mass value="1e-5" />
-      <origin xyz="0 0 0" rpy="0 0 0"/>
-      <inertia ixx="1e-6" ixy="0" ixz="0" iyy="1e-6" iyz="0"      izz="1e-6" />
-    </inertial>
-  </link>
-  <joint name="sonar_front_joint" type="fixed">
-    <axis xyz="0 1 0" />
-    <origin rpy="0 0 0" xyz="0.02 0 0.1" />
-    <parent link="${namespace}/base_link"/>
-    <child link="base_sonar_front_0"/>
-  </joint>
-  <link name="base_sonar_front_0">
-    <collision>
-      <origin xyz="0 0 0" rpy="0 0 0"/>
-      <geometry>
-        <box size="0.01 0.01 0.01"/>
-      </geometry>
-    </collision>
-    <visual>
-      <origin xyz="0 0 0" rpy="0 0 0"/>
-      <geometry>
-        <box size="0.01 0.01 0.01"/>
-      </geometry>
-    </visual>
-    <inertial>
-      <mass value="1e-5" />
-      <origin xyz="0 0 0" rpy="0 0 0"/>
-      <inertia ixx="1e-6" ixy="0" ixz="0" iyy="1e-6" iyz="0" izz="1e-6" />
-    </inertial>
-  </link>
-  <joint name="ir_front_joint_45" type="fixed">
-    <axis xyz="0 1 0" />
-    <origin rpy="0 0 0.78539816339" xyz="0.01 0.01 0.1" />
-    <parent link="${namespace}/base_link"/>
-    <child link="base_ir_front_45"/>
-  </joint>
-  <link name="base_ir_front_45">
-    <collision>
-      <origin xyz="0 0 0" rpy="0 0 0"/>
-      <geometry>
-        <box size="0.01 0.01 0.01"/>
-      </geometry>
-    </collision>
-    <visual>
-      <origin xyz="0 0 0" rpy="0 0 0"/>
-      <geometry>
-        <box size="0.01 0.01 0.01"/>
-      </geometry>
-    </visual>
-    <inertial>
-      <mass value="1e-5" />
-      <origin xyz="0 0 0" rpy="0 0 0"/>
-      <inertia ixx="1e-6" ixy="0" ixz="0" iyy="1e-6" iyz="0"      izz="1e-6" />
-    </inertial>
-  </link>
-  <joint name="sonar_front_joint_45" type="fixed">
-    <axis xyz="0 1 0" />
-    <origin rpy="0 0 0.78539816339" xyz="0.01 0.01 0.1" />
-    <parent link="${namespace}/base_link"/>
-    <child link="base_sonar_front_45"/>
-  </joint>
-  <link name="base_sonar_front_45">
-    <collision>
-      <origin xyz="0 0 0" rpy="0 0 0"/>
-      <geometry>
-        <box size="0.01 0.01 0.01"/>
-      </geometry>
-    </collision>
-    <visual>
-      <origin xyz="0 0 0" rpy="0 0 0"/>
-      <geometry>
-        <box size="0.01 0.01 0.01"/>
-      </geometry>
-    </visual>
-    <inertial>
-      <mass value="1e-5" />
-      <origin xyz="0 0 0" rpy="0 0 0"/>
-      <inertia ixx="1e-6" ixy="0" ixz="0" iyy="1e-6" iyz="0" izz="1e-6" />
-    </inertial>
-  </link>
-  <joint name="ir_front_joint_90" type="fixed">
-    <axis xyz="0 1 0" />
-    <origin rpy="0 0 1.57079632679" xyz="0.0 0.02 0.1" />
-    <parent link="${namespace}/base_link"/>
-    <child link="base_ir_front_90"/>
-  </joint>
-  <link name="base_ir_front_90">
-    <collision>
-      <origin xyz="0 0 0" rpy="0 0 0"/>
-      <geometry>
-        <box size="0.01 0.01 0.01"/>
-      </geometry>
-    </collision>
-    <visual>
-      <origin xyz="0 0 0" rpy="0 0 0"/>
-      <geometry>
-        <box size="0.01 0.01 0.01"/>
-      </geometry>
-    </visual>
-    <inertial>
-      <mass value="1e-5" />
-      <origin xyz="0 0 0" rpy="0 0 0"/>
-      <inertia ixx="1e-6" ixy="0" ixz="0" iyy="1e-6" iyz="0"      izz="1e-6" />
-    </inertial>
-  </link>
-  <joint name="sonar_front_joint_90" type="fixed">
-    <axis xyz="0 1 0" />
-    <origin rpy="0 0 1.57079632679" xyz="0. 0.02 0.1" />
-    <parent link="${namespace}/base_link"/>
-    <child link="base_sonar_front_90"/>
-  </joint>
-  <link name="base_sonar_front_90">
-    <collision>
-      <origin xyz="0 0 0" rpy="0 0 0"/>
-      <geometry>
-        <box size="0.01 0.01 0.01"/>
-      </geometry>
-    </collision>
-    <visual>
-      <origin xyz="0 0 0" rpy="0 0 0"/>
-      <geometry>
-        <box size="0.01 0.01 0.01"/>
-      </geometry>
-    </visual>
-    <inertial>
-      <mass value="1e-5" />
-      <origin xyz="0 0 0" rpy="0 0 0"/>
-      <inertia ixx="1e-6" ixy="0" ixz="0" iyy="1e-6" iyz="0" izz="1e-6" />
-    </inertial>
-  </link>
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